Commit message: Aumentar resolucion del LIDAR a 720 rayos + segundo mundo depot.world
- LIDAR: samples 360->720 (resolution se mantiene en 1, o sea ahora son
  720 rayos reales en vez de 360, ~0.5 grados entre rayo y rayo).
- Ajuste de castor_wheel_collision_radius 0.0125->0.0225.
- Nuevo mundo depot.world (deposito de Open Robotics via Fuel, sin el
  robot Tugbot que traia incluido) como segundo mundo de la Parte 1.
- Mapas guardados: depot.pgm/.yaml (nuevo) y living_room.pgm/.yaml
  actualizado (remapeado).

Co-Authored-By: Claude Sonnet 5 <noreply@anthropic.com>

File: TP2-Grupo7/src/my_robot_description/urdf/mobile_base.xacro (robot description, xacro)
@@ -49,5 +49,5 @@
   <xacro:property name="wheel_collision_radius" value="0.033"/>
   <xacro:property name="wheel_collision_length" value="0.020"/>
-  <xacro:property name="castor_wheel_collision_radius" value="0.0125"/>
+  <xacro:property name="castor_wheel_collision_radius" value="0.0225"/>
   <xacro:property name="lidar_collision_radius" value="0.03"/>
   <xacro:property name="lidar_collision_length" value="0.04"/>
@@ -308,5 +308,5 @@
         <scan>
           <horizontal>
-            <samples>360</samples>
+            <samples>720</samples>
             <resolution>1</resolution>
             <min_angle>-3.141592</min_angle>
